File: hw_rev1/kicad/ProPrj_SPE 10BASE-T1L USB adapter.kicad_pcb (KiCad board)
At the start: 4 copper layers, 22 x 51.5 mm, 75 parts

Commit message: Add KiCad design rules file + cleanup DRC
Routing:
- net 3V3: vias 17 -> 16

Commit message: Cleanup KiCad schematic
Parts:
- C1, C2: value (none) -> 100pF
- C13, C14: value (none) -> 10uF
- C15, C16: value (none) -> 15pF
- C17, C18: value (none) -> 33pF
- C19, C20, C21, C22, C23, C24, C25, C26, C27, C28, C29, C32, C36: value (none) -> 100nF
- C3, C4: value (none) -> 220nF
- C30, C33, C37: value (none) -> 1uF
- C31, C34, C35: value (none) -> 10nF
- D8: value (none) -> USBLC6-2SC6
- D9: value (none) -> SRF0905A-471Y
- L1, L2, L3, L4: value (none) -> BLM15PD121SN1D
- LED1, LED2: value (none) -> KT-0603R
- P1: value (none) -> WJ15EDGRC-3.81-02P-14-00A
- Q1: value (none) -> LBSS84LT1G
- R1, R4: value (none) -> 50Ω
- R100, R101, R87, R99: value (none) -> 10kΩ
- R102, R97, R98: value (none) -> 2.49kΩ
- R2, R3: value (none) -> 2kΩ
- R40, R41: value (none) -> 5.1kΩ
- R5: value (none) -> 470kΩ
- R84: value (none) -> 47Ω
- R85, R86: value (none) -> 12kΩ
- R88, R89: value (none) -> 1kΩ
- R95: value (none) -> 499Ω
- R96: value (none) -> 2.2kΩ
- TP1, TP2, TP3, TP4: renamed from ?; value (none) -> TestPoint
- U1: value (none) -> LAN9500A-ABZJ-TR
- U2: value (none) -> DP83TD510ERHBR
- U3: value (none) -> PESD2ETH-AXR
- U6: value (none) -> RT9080-33GJ5
- USB2: value (none) -> TYPE-C 16PIN 2MD(073)
- X1, X2: value (none) -> 25MHz
Connections:
- net $1N11057 renamed Net-(Q1-D)
- net $1N1869 renamed Net-(X1-OSC1)
- net $1N1960 renamed Net-(X2-OSC1)
- net $1N2873 renamed Net-(U1-USBRBIAS)
- net $1N3850 renamed Net-(U1-EXRES)
- net $1N4408 renamed Net-(LED1-A)
- net $1N4707 renamed Net-(LED2-A)
- net $1N5728 renamed Net-(C3-Pad1)
- net $1N5733 renamed Net-(C4-Pad1)
- net $1N5739 renamed Net-(C3-Pad2)
- net $1N5745 renamed Net-(C4-Pad2)
- net $1N5759 renamed Net-(C1-Pad2)
- net $1N5765 renamed Net-(C2-Pad2)
- net MAC_AVDD renamed /MAC_AVDD
- net MAC_COL renamed /MAC_COL
- net MAC_CRS renamed /MAC_CRS
- net MAC_NRST renamed /MAC_NRST
- net MAC_PHYSEL renamed /MAC_PHYSEL
- net MAC_VDDCORE renamed /MAC_VDDCORE
- net MAC_VDDPLL renamed /MAC_VDDPLL
- net MAC_VDDUSB renamed /MAC_VDDUSB
- net MAC_XI renamed /MAC_XI
- net MAC_XO renamed /MAC_XO
- net MDC renamed /MDC
- net MDIO renamed /MDIO
- net PHY_DVDD renamed /PHY_DVDD
- net PHY_INT renamed /PHY_INT
- net PHY_IO2 renamed /PHY_IO2
- net PHY_LED0 renamed /PHY_LED0
- net PHY_RST renamed /PHY_RST
- net PHY_VDDA renamed /PHY_VDDA
- net PHY_XI renamed /PHY_XI
- net PHY_XO renamed /PHY_XO
- net RXCLK renamed /RXCLK
- net RXD0 renamed /RXD0
- net RXD1 renamed /RXD1
- net RXD2 renamed /RXD2
- net RXD3 renamed /RXD3
- net RXDV renamed /RXDV
- net RXER renamed /RXER
- net RXN renamed /RXN
- net RXP renamed /RXP
- net TXCLK renamed /TXCLK
- net TXD0 renamed /TXD0
- net TXD1 renamed /TXD1
- net TXD2 renamed /TXD2
- net TXD3 renamed /TXD3
- net TXEN renamed /TXEN
- net TXN renamed /TXN
- net TXP renamed /TXP
- net USB_CC1 renamed /USB_CC1
- net USB_CC2 renamed /USB_CC2
- net USB_DN renamed /USB_DN
- net USB_DN_C renamed /USB_DN_C
- net USB_DP renamed /USB_DP
- net USB_DP_C renamed /USB_DP_C
- U1 pad 14: (no net) -> unconnected-(U1-NC-Pad14)
- U1 pad 2: (no net) -> unconnected-(U1-TXN-Pad2)
- U1 pad 26: (no net) -> unconnected-(U1-nFDX_LED/GPIO8-Pad26)
- U1 pad 27: (no net) -> unconnected-(U1-nLNKA_LED/GPIO9-Pad27)
- U1 pad 28: (no net) -> unconnected-(U1-nSPD_LED/GPIO10-Pad28)
- U1 pad 29: (no net) -> unconnected-(U1-EECLK/PWR_SEL-Pad29)
- U1 pad 3: (no net) -> unconnected-(U1-TXP-Pad3)
- U1 pad 30: (no net) -> unconnected-(U1-EECS-Pad30)
- U1 pad 31: (no net) -> unconnected-(U1-EEDO/AUTOMDIX_EN-Pad31)
- U1 pad 32: (no net) -> unconnected-(U1-EEDI-Pad32)
- U1 pad 5: (no net) -> unconnected-(U1-RXN-Pad5)
- U1 pad 6: (no net) -> unconnected-(U1-RXP-Pad6)
- U2 pad 28: (no net) -> unconnected-(U2-LED_2/TX_ER/Strap7-Pad28)
- U2 pad 30: (no net) -> unconnected-(U2-CLKOUT/LED_1-Pad30)
- U2 pad 32: (no net) -> unconnected-(U2-GPIO1/Strap9-Pad32)
- U3 pad 4: (no net) -> unconnected-(U3-Pad4)
- U6 pad 4: (no net) -> unconnected-(U6-NC-Pad4)
- USB2 pad 3: (no net) -> unconnected-(USB2-SBU2-Pad3)
- USB2 pad 9: (no net) -> unconnected-(USB2-SBU1-Pad9)
- X1 pad 2: (no net) -> unconnected-(X1-GND-Pad2)
- X1 pad 4: (no net) -> unconnected-(X1-GND-Pad4)
- X2 pad 2: (no net) -> unconnected-(X2-GND-Pad2)
- X2 pad 4: (no net) -> unconnected-(X2-GND-Pad4)
