File: hw_rev1/kicad/ProPrj_SPE 10BASE-T1L USB adapter.kicad_sch (KiCad schematic)
At the start: 67 parts, among them P1 WJ15EDGRC-3.81-02P-14-00A, Q1 LBSS84LT1G, U1 LAN9500A-ABZJ-TR, U2 DP83TD510ERHBR, U3 PESD2ETH-AXR, U6 RT9080-33GJ5, X1 25MHz, X2 25MHz

Commit message: Cleanup KiCad schematic
Parts:
- added TP1: TestPoint, ProPrj_SPE 10BASE-T1L USB adapter:Pad_e105, symbol ProPrj_SPE-easyedapro:TestPoint
- added TP2: TestPoint, ProPrj_SPE 10BASE-T1L USB adapter:Pad_e106, symbol ProPrj_SPE-easyedapro:TestPoint
- added TP3: TestPoint, ProPrj_SPE 10BASE-T1L USB adapter:Pad_e107, symbol ProPrj_SPE-easyedapro:TestPoint
- added TP4: TestPoint, ProPrj_SPE 10BASE-T1L USB adapter:Pad_e108, symbol ProPrj_SPE-easyedapro:TestPoint
- C1, C13, C14, C2: footprint ProPrj_SPE-easyedapro:C0603 -> ProPrj_SPE 10BASE-T1L USB adapter:C0603
- C15, C16, C17, C18, C19, C20, C21, C22, C23, C24, C25, C26, C27, C28, C29, C30, C31, C32, C33, C34, C35, C36, C37: footprint ProPrj_SPE-easyedapro:C0402 -> ProPrj_SPE 10BASE-T1L USB adapter:C0402
- C3, C4: footprint ProPrj_SPE-easyedapro:C0805 -> ProPrj_SPE 10BASE-T1L USB adapter:C0805
- D8: footprint ProPrj_SPE-easyedapro:SOT-23-6_L2.9-W1.6-P0.95-LS2.8-BL -> ProPrj_SPE 10BASE-T1L USB adapter:SOT-23-6_L2.9-W1.6-P0.95-LS2.8-BL
- D9: footprint ProPrj_SPE-easyedapro:FILTER-SMD_4P-L9.2-W6.0-TL-A -> ProPrj_SPE 10BASE-T1L USB adapter:FILTER-SMD_4P-L9.2-W6.0-TL-A
- L1, L2, L3, L4: footprint ProPrj_SPE-easyedapro:L0402 -> ProPrj_SPE 10BASE-T1L USB adapter:L0402
- LED1, LED2: footprint ProPrj_SPE-easyedapro:LED-SMD_L1.6-W0.8-R-RD -> ProPrj_SPE 10BASE-T1L USB adapter:LED-SMD_L1.6-W0.8-R-RD
- P1: footprint ProPrj_SPE-easyedapro:CONN-TH_2P-P3.81_WJ15EDGRC-3.81-2P -> ProPrj_SPE 10BASE-T1L USB adapter:CONN-TH_2P-P3.81_WJ15EDGRC-3.81-2P
- Q1: footprint ProPrj_SPE-easyedapro:SOT-23_L2.9-W1.3-P1.90-LS2.4-BR -> ProPrj_SPE 10BASE-T1L USB adapter:SOT-23_L2.9-W1.3-P1.90-LS2.4-BR
- R1, R2, R3, R4: footprint ProPrj_SPE-easyedapro:R0603 -> ProPrj_SPE 10BASE-T1L USB adapter:R0603
- R100, R101, R102, R40, R41, R5, R84, R85, R86, R87, R88, R89, R95, R96, R97, R98, R99: footprint ProPrj_SPE-easyedapro:R0402 -> ProPrj_SPE 10BASE-T1L USB adapter:R0402
- U1: footprint ProPrj_SPE-easyedapro:QFN-56_L8.0-W8.0-P0.50-TL-EP6.1 -> ProPrj_SPE 10BASE-T1L USB adapter:QFN-56_L8.0-W8.0-P0.50-TL-EP6.1
- U2: footprint ProPrj_SPE-easyedapro:HVQFN-32_L5.0-W5.0-P0.50-TL-EP2.1 -> ProPrj_SPE 10BASE-T1L USB adapter:HVQFN-32_L5.0-W5.0-P0.50-TL-EP2.1
- U3: footprint ProPrj_SPE-easyedapro:SOT-143_L2.9-W1.3-P1.92-LS2.3-BL -> ProPrj_SPE 10BASE-T1L USB adapter:SOT-143_L2.9-W1.3-P1.92-LS2.3-BL
- U6: footprint ProPrj_SPE-easyedapro:TSOT-23-5_L2.9-W1.6-P0.95-LS2.8-BL -> ProPrj_SPE 10BASE-T1L USB adapter:TSOT-23-5_L2.9-W1.6-P0.95-LS2.8-BL
- USB2: footprint ProPrj_SPE-easyedapro:USB-C-SMD_TYPE-C-6PIN-2MD-073 -> ProPrj_SPE 10BASE-T1L USB adapter:USB-C-SMD_TYPE-C-6PIN-2MD-073
- X1: footprint ProPrj_SPE-easyedapro:CRYSTAL-SMD_4P-L3.2-W2.5-BL -> ProPrj_SPE 10BASE-T1L USB adapter:CRYSTAL-SMD_4P-L3.2-W2.5-BL
- X2: footprint ProPrj_SPE-easyedapro:CRYSTAL-SMD_4P-L3.2-W2.5-BL-2 -> ProPrj_SPE 10BASE-T1L USB adapter:CRYSTAL-SMD_4P-L3.2-W2.5-BL-2
Connections:
- net 3V3: now also TP3.1
- net MDC: now also TP2.1
- net MDIO: now also TP1.1
- net USB_DP: now also D8.4 (IO2)
- net VCC5V0_SYS: now also TP4.1; no longer D8.4 (IO2)
- no-connect marks 18 -> 22
Other:
- moved on the sheet: C13, C14, LED2, R89
